File: hardware_controle.kicad_sch (KiCad schematic)
At the start: 19 parts, among them J10 JP LED, J7 FB TRANCA, J8 Con. Placa Aux., J9 Con. Alimentação 9.5V, U2 NE555P

Commit message: Add files via upload
Parts:
- removed J8: Con. Placa Aux., Connector_PinHeader_2.54mm:PinHeader_1x08_P2.54mm_Vertical, symbol Connector:Conn_01x08_Male
- added J1: Con. Placa Aux., Connector_PinHeader_2.54mm:PinHeader_1x09_P2.54mm_Vertical, symbol Connector_Generic:Conn_01x09
- J7: footprint TerminalBlock_MetzConnect:TerminalBlock_MetzConnect_360381_1x01_Horizontal_ScrewM3.0 -> TerminalBlock_RND:TerminalBlock_RND_205-00012_1x02_P5.00mm_Horizontal
- J9: footprint TerminalBlock_Phoenix:TerminalBlock_Phoenix_MPT-0,5-2-2.54_1x02_P2.54mm_Horizontal -> TerminalBlock_RND:TerminalBlock_RND_205-00012_1x02_P5.00mm_Horizontal
Connections:
- net +5: now also J1.1 (Pin_1)
- net 3.3v: now also J1.2 (Pin_2)
- net CE: now also J1.7 (Pin_7)
- net GND: now also J1.9 (Pin_9)
- net MISO: now also J1.5 (Pin_5)
- net MOSI: now also J1.6 (Pin_6)
- net RST: now also J1.8 (Pin_8)
- net SCLK: now also J1.4 (Pin_4)
- net TR_CNTRL: now also J1.3 (Pin_3)
- net contato_porta: now reaches J7.1 (Pin_1), R1.1
Changed lines of the file:
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@@
+    (stroke (width 0) (type default) (color 0 0 0 0))
+  )
+  (wire (pts (xy 203.2 46.99) (xy 207.01 46.99))
     (stroke (width 0) (type default) (color 0 0 0 0))
   )
@@
     (stroke (width 0) (type default) (color 0 0 0 0))
   )
-  (polyline (pts (xy 267.97 69.85) (xy 267.97 45.72))
+  (polyline (pts (xy 267.97 69.85) (xy 267.97 40.64))
     (stroke (width 0) (type default) (color 0 0 0 0))
   )
@@
     (stroke (width 0) (type default) (color 0 0 0 0))
   )
-  (polyline (pts (xy 267.97 45.72) (xy 185.42 45.72))
-    (stroke (width 0) (type default) (color 0 0 0 0))
-  )
-  (polyline (pts (xy 185.42 45.72) (xy 185.42 69.85))
+  (polyline (pts (xy 267.97 40.64) (xy 185.42 40.64))
+    (stroke (width 0) (type default) (color 0 0 0 0))
+  )
+  (polyline (pts (xy 185.42 40.64) (xy 185.42 69.85))
     (stroke (width 0) (type default) (color 0 0 0 0))
   )
@@
     (effects (font (size 1.27 1.27)) (justify left bottom))
   )
-  (text "CONEXÕES BARRA DE PINOS" (at 213.36 45.72 0)
+  (text "CONEXÕES BARRA DE PINOS" (at 215.9 40.64 0)
     (effects (font (size 1.27 1.27)) (justify left bottom))
   )
@@
   )
   (text "PROTEÇÃO DA ALIMENTAÇÃO" (at 39.37 25.4 0)
+    (effects (font (size 1.27 1.27)) (justify left bottom))
+  )
+  (label "contato_porta" (at 43.18 85.09 90)
     (effects (font (size 1.27 1.27)) (justify left bottom))
   )
@@
     (property "Reference" "J9" (id 0) (at 30.48 36.83 90))
     (property "Value" "Con. Alimentação 9.5V" (id 1) (at 33.02 36.83 90))
-    (property "Footprint" "TerminalBlock_Phoenix:TerminalBlock_Phoenix_MPT-0,5-2-2.54_1x02_P2.54mm_Horizontal" (id 2) (at 35.56 35.56 0)
+    (property "Footprint" "TerminalBlock_RND:TerminalBlock_RND_205-00012_1x02_P5.00mm_Horizontal" (id 2) (at 35.56 35.56 0)
       (effects (font (size 1.27 1.27)) hide)
     )
@@
     (pin "6")
     (pin "7")
+  )
+  (symbol (lib_id "Connector_Generic:Conn_01x09") (at 212.09 57.15 0) (mirror x) (unit 1)
+    (in_bom yes) (on_board yes)
+    (property "Reference" "J1" (id 0) (at 217.17 62.23 90))
+    (property "Value" "Con. Placa Aux." (id 1) (at 214.63 60.96 90))
+    (property "Footprint" "Connector_PinHeader_2.54mm:PinHeader_1x09_P2.54mm_Vertical" (id 2) (at 212.09 57.15 0)
+      (effects (font (size 1.27 1.27)) hide)
+    )
+    (property "Datasheet" "~" (id 3) (at 212.09 57.15 0)
+      (effects (font (size 1.27 1.27)) hide)
+    )
+    (pin "1")
+    (pin "2")
+    (pin "3")
+    (pin "4")
+    (pin "5")
+    (pin "6")
+    (pin "7")
+    (pin "8")
+    (pin "9")
   )
   (symbol (lib_id "power:GND") (at 220.98 137.16 0) (unit 1)
@@
     (pin "2")
   )
+  (symbol (lib_id "power:GND") (at 203.2 46.99 180) (unit 1)
+    (in_bom yes) (on_board yes)
+    (property "Reference" "#PWR07" (id 0) (at 203.2 40.64 0)
+      (effects (font (size 1.27 1.27)) hide)
+    )
+    (property "Value" "GND" (id 1) (at 203.2 43.18 0))
+    (property "Footprint" "" (id 2) (at 203.2 46.99 0)
+      (effects (font (size 1.27 1.27)) hide)
+    )
+    (property "Datasheet" "" (id 3) (at 203.2 46.99 0)
+      (effects (font (size 1.27 1.27)) hide)
+    )
+    (pin "1")
+  )
   (symbol (lib_id "Device:R") (at 52.07 85.09 90) (unit 1)
     (in_bom yes) (on_board yes) (fields_autoplaced)
@@
     (property "Reference" "J7" (id 0) (at 38.1 82.55 0))
     (property "Value" "FB TRANCA" (id 1) (at 39.37 87.63 0))
-    (property "Footprint" "TerminalBlock_MetzConnect:TerminalBlock_MetzConnect_360381_1x01_Horizontal_ScrewM3.0" (id 2) (at 38.1 85.09 0)
+    (property "Footprint" "TerminalBlock_RND:TerminalBlock_RND_205-00012_1x02_P5.00mm_Horizontal" (id 2) (at 38.1 85.09 0)
       (effects (font (size 1.27 1.27)) hide)
     )
@@
     )
     (pin "1")
-  )
-  (symbol (lib_id "Connector:Conn_01x08_Male") (at 212.09 59.69 180) (unit 1)
-    (in_bom yes) (on_board yes)
-    (property "Reference" "J8" (id 0) (at 215.9 58.42 90)
-      (effects (font (size 1.27 1.27)) (justify right))
-    )
-    (property "Value" "Con. Placa Aux." (id 1) (at 213.36 64.77 90)
-      (effects (font (size 1.27 1.27)) (justify right))
-    )
-    (property "Footprint" "Connector_PinHeader_2.54mm:PinHeader_1x08_P2.54mm_Vertical" (id 2) (at 212.09 59.69 0)
-      (effects (font (size 1.27 1.27)) hide)
-    )
-    (property "Datasheet" "~" (id 3) (at 212.09 59.69 0)
-      (effects (font (size 1.27 1.27)) hide)
-    )
-    (pin "1")
-    (pin "2")
-    (pin "3")
-    (pin "4")
-    (pin "5")
-    (pin "6")
-    (pin "7")
-    (pin "8")
   )
   (symbol (lib_id "Device:R") (at 40.64 138.43 90) (unit 1)
@@
       (reference "#PWR06") (unit 1) (value "GND") (footprint "")
     )
+    (path "/94c0495a-6eab-4dcc-bcae-6f1e92a1c88a"
+      (reference "#PWR07") (unit 1) (value "GND") (footprint "")
+    )
     (path "/f9c11e37-75a2-4d86-8e9e-14c863c69730"
       (reference "#PWR011") (unit 1) (value "GND") (footprint "")
@@
       (reference "D3") (unit 1) (value "DIODE") (footprint "Diode_THT:D_DO-41_SOD81_P7.62mm_Horizontal")
     )
+    (path "/725a4702-9d8d-41c5-99fe-07f4d5771c53"
+      (reference "J1") (unit 1) (value "Con. Placa Aux.") (footprint "Connector_PinHeader_2.54mm:PinHeader_1x09_P2.54mm_Vertical")
+    )
     (path "/9a492cdc-3b73-47b9-bed1-f8fff4d88818"
-      (reference "J7") (unit 1) (value "FB TRANCA") (footprint "TerminalBlock_MetzConnect:TerminalBlock_MetzConnect_360381_1x01_Horizontal_ScrewM3.0")
-    )
-    (path "/c8698a49-36d6-44b5-93ec-98b5332f1eda"
-      (reference "J8") (unit 1) (value "Con. Placa Aux.") (footprint "Connector_PinHeader_2.54mm:PinHeader_1x08_P2.54mm_Vertical")
+      (reference "J7") (unit 1) (value "FB TRANCA") (footprint "TerminalBlock_RND:TerminalBlock_RND_205-00012_1x02_P5.00mm_Horizontal")
     )
     (path "/3df25e06-8787-4e1a-ba1c-db1644863894"
-      (reference "J9") (unit 1) (value "Con. Alimentação 9.5V") (footprint "TerminalBlock_Phoenix:TerminalBlock_Phoenix_MPT-0,5-2-2.54_1x02_P2.54mm_Horizontal")
+      (reference "J9") (unit 1) (value "Con. Alimentação 9.5V") (footprint "TerminalBlock_RND:TerminalBlock_RND_205-00012_1x02_P5.00mm_Horizontal")
     )
     (path "/1207cfb3-2dab-4b69-ae32-dc83052f265e"
